Commit message: update

File: urdf/actuator.xacro (robot description, xacro)
@@ -1,4 +1,4 @@
 <?xml version="1.0"?>
-<robot>
+<robot xmlns:xacro="http://ros.org/wiki/xacro">
   <!-- front steering -->
   <transmission name="steering_left_front_trans">

File: urdf/steering.xacro (robot description, xacro)
@@ -1,2 +1,3 @@
+<?xml version="1.0"?>
 <robot xmlns:xacro="http://ros.org/wiki/xacro">
   <xacro:property name="pi" value="3.1415926835897931" />
@@ -7,13 +8,12 @@
       <child  link="${suffix}_link"/>
       <axis xyz="0 0 1"/>
-      <limit effort="1000.0" lower="-1" upper="1" velocity="0.5"/>
+      <limit effort="1000.0" lower="-0.6" upper="0.6" velocity="0.5"/>
     </joint>
     <link name="${suffix}_link">
       <visual>
         <geometry>
-          <box size="0.01 0.01 0.01"/>
-          <!-- <cylinder length="0.01" radius="0.1"/> -->
+          <cylinder radius="0.1" length="0.01"/>
         </geometry>
-        <origin xyz="0 0 0" rpy="0 0 0"/>
+        <origin xyz="0 0 0" rpy="${pi/2} 0 0"/>
         <material name="black">
           <color rgba="0.1 0.1 0.1 2.0"/>
@@ -22,34 +22,16 @@
       <inertial>
         <origin xyz="0 0 0" rpy="0 0 0"/>
-        <mass value="0.01"/>
-        <inertia ixx="${(0.0001+0.0001)*0.01/12}"  ixy="0"  ixz="0" iyy="${(0.0001+0.0001)*0.01/12}" iyz="0" izz="${(0.0001+0.0001)*0.01/12}" />
+        <mass value="10.0"/>
+        <inertia ixx="0.0250833"  ixy="0"  ixz="0" iyy="0.05" iyz="0" izz="0.0250833" />
+        <!-- <mass value="10.0"/>
+        <inertia ixx="0.4"  ixy="0"  ixz="0" iyy="0.6" iyz="0" izz="0.4" /> -->
       </inertial>
-      <collision>
-        <origin xyz="0 0 0" rpy="0 0 0"/>
+      <!-- <collision>
+        <origin xyz="0 0 0" rpy="${pi/2} 0 0"/>
         <geometry>
-          <box size="0.01 0.01 0.01"/>
-          <!-- <cylinder radius="0.1" length="0.01" /> -->
+          <cylinder radius="0.1" length="0.01" />
         </geometry>
-      </collision>
+      </collision> -->
     </link>
-    <!-- <transmission name="${suffix}_trans">
-      <type>transmission_interface/SimpleTransmission</type>
-      <joint name="${suffix}_joint">
-        <hardwareInterface>hardware_interface/PositionJointInterface</hardwareInterface>
-      </joint>
-      <actuator name="${suffix}_motor">
-         <hardwareInterface>hardware_interface/PositionJointInterface</hardwareInterface>
-         <mechanismReduction>1</mechanismReduction>
-      </actuator>
-    </transmission> -->
-    <!-- <gazebo reference="${suffix}_link">
-      <material>Gazebo/Red</material>
-        <mu1 value="0.6" />
-        <mu2 value="0.5" />
-        <kp value="1000000" />
-        <kd value="0.1" />
-        <minDepth value="0.01"/>
-        <maxVel value="10.0" />
-    </gazebo> -->
   </xacro:macro>
 </robot>

File: urdf/vehicle.xacro (robot description, xacro)
@@ -1,3 +1,5 @@
+<?xml version="1.0"?>
 <robot name="autoware" xmlns:xacro="http://ros.org/wiki/xacro">
+  <xacro:include filename="$(find vehicle_model)/urdf/body.xacro" />
   <xacro:include filename="$(find vehicle_model)/urdf/wheel.xacro" />
   <xacro:include filename="$(find vehicle_model)/urdf/steering.xacro" />
@@ -11,32 +13,15 @@
   <xacro:arg name="vehicle_height" default="1.5"/>
   <xacro:arg name="vehicle_mass_height" default="0.5"/>
-  <xacro:property name="pi" value="3.1415926835897931" />
+  <xacro:property name="pi" value="3.1415926835897931"/>
   <link name="base_link"/>
-  <joint name="base_joint" type="fixed">
-    <parent link="base_link"/>
-    <origin rpy="0 0 0" xyz="0 0 $(arg wheel_radius)"/>
-    <child  link="wheel_base_link"/>
-  </joint>
-  <link name="wheel_base_link">
-    <inertial>
-      <origin xyz="${$(arg wheel_base)/2} 0 0" rpy="0 0 0"/>
-      <mass value="$(arg vehicle_mass)"/>
-      <inertia ixx="${($(arg vehicle_width)*$(arg vehicle_width)+$(arg vehicle_mass_height)*$(arg vehicle_mass_height))*$(arg vehicle_mass)/12.0}" ixy="0.0" ixz="0.0"
-               iyy="${($(arg vehicle_length)*$(arg vehicle_length)+$(arg vehicle_mass_height)*$(arg vehicle_mass_height))*$(arg vehicle_mass)/12.0}" iyz="0.0"
-               izz="${($(arg vehicle_width)*$(arg vehicle_width)+$(arg vehicle_length)*$(arg vehicle_length))*$(arg vehicle_mass)/12.0}"/>
-    </inertial>
-    <visual>
-      <origin xyz="${$(arg wheel_base)/2} 0 ${$(arg vehicle_height)/2}" rpy="0 0 0"/>
-      <geometry>
-        <box size="$(arg vehicle_length) $(arg vehicle_width) $(arg vehicle_height)"/>
-      </geometry>
-    </visual>
-    <collision>
-      <origin xyz="${$(arg wheel_base)/2} 0 ${$(arg vehicle_height)/2}" rpy="0 0 0"/>
-      <geometry>
-        <box size="$(arg vehicle_length) 0.9 $(arg vehicle_height)"/>
-      </geometry>
-    </collision>
-  </link>
+  <xacro:body_macro suffix="wheel_base"
+                    parent="base_link"
+                    wheel_radius="$(arg wheel_radius)"
+                    wheel_base="$(arg wheel_base)"
+                    vehicle_mass="$(arg vehicle_mass)"
+                    vehicle_mass_height="$(arg vehicle_mass_height)"
+                    vehicle_length="$(arg vehicle_length)"
+                    vehicle_width="$(arg vehicle_width)"
+                    vehicle_height="$(arg vehicle_height)"/>
   <xacro:steering_macro suffix="steering_right_front" parent="wheel_base_link" x="$(arg wheel_base)" y="${-1*$(arg wheel_tread)/2}" yaw="0" length="$(arg wheel_width)"/>
   <xacro:steering_macro suffix="steering_left_front" parent="wheel_base_link" x="$(arg wheel_base)" y="${$(arg wheel_tread)/2}" yaw="0" length="$(arg wheel_width)"/>
@@ -50,19 +35,4 @@
  	<xacro:include filename="$(find vehicle_model)/urdf/actuator.xacro"/>
   <!-- gazebo -->
- 	<xacro:include filename="$(find vehicle_model)/urdf/wheel.gazebo"/>
- 	<xacro:include filename="$(find vehicle_model)/urdf/steering.gazebo"/>
-  <gazebo>
-    <plugin name="gazebo_ros_control" filename="libgazebo_ros_control.so">
-      <robotNamespace>/autoware</robotNamespace>
-      <robotSimType>gazebo_ros_control/DefaultRobotHWSim</robotSimType>
-    </plugin>
-  </gazebo>
-  <gazebo>
-    <plugin filename="libgazebo_ros_joint_state_publisher.so" name="joint_state_publisher">
-      <jointName>wheel_left_rear_joint, wheel_right_rear_joint, steering_left_front_joint, steering_right_front_joint</jointName>
-      <updateRate>50.0</updateRate>
-      <robotNamespace>/autoware</robotNamespace>
-      <alwaysOn>true</alwaysOn>
-    </plugin>
-  </gazebo>
+ 	<xacro:include filename="$(find vehicle_model)/urdf/vehicle.gazebo"/>
 </robot>

File: urdf/wheel.xacro (robot description, xacro)
@@ -1,2 +1,3 @@
+<?xml version="1.0"?>
 <robot xmlns:xacro="http://ros.org/wiki/xacro">
   <xacro:property name="pi" value="3.1415926835897931" />
@@ -34,23 +35,4 @@
       </collision>
     </link>
-    <!-- <transmission name="${suffix}_trans">
-      <type>transmission_interface/SimpleTransmission</type>
-      <joint name="${suffix}_joint">
-        <hardwareInterface>hardware_interface/VelocityJointInterface</hardwareInterface>
-      </joint>
-      <actuator name="${suffix}_motor">
-         <hardwareInterface>hardware_interface/VelocityJointInterface</hardwareInterface>
-         <mechanismReduction>1</mechanismReduction>
-      </actuator>
-    </transmission> -->
-    <!-- <gazebo reference="${suffix}_link">
-      <material>Gazebo/Red</material>
-      <mu1 value="10000.0" />
-      <mu2 value="10000.0" />
-   		<kp value="100000" />
-      <kd value="0.1" />
-      <minDepth value="0.01" />
-      <maxVel  value="100.0" />
-    </gazebo> -->
   </xacro:macro>
 </robot>
