Commit message: update

File: urdf/body.xacro (robot description, xacro)
@@ -17,4 +17,13 @@
       </inertial>
       <visual>
+        <origin xyz="${wheel_base/2} 0 ${vehicle_height/2}" rpy="0 ${-pi/2} ${pi/2}"/>
+        <geometry>
+          <mesh filename="package://vehicle_model/dae/banana.dae" scale="0.7 0.7 0.7"/>
+        </geometry>
+        <material name="black">
+            <color rgba="0.1 0.1 0.1 2.0"/>
+        </material>
+      </visual>
+      <!-- <visual>
         <origin xyz="${wheel_base/2} 0 ${vehicle_height/2}" rpy="0 0 0"/>
         <geometry>
@@ -24,5 +33,5 @@
             <color rgba="0.1 0.1 0.1 2.0"/>
         </material>
-      </visual>
+      </visual> -->
       <collision>
         <origin xyz="${wheel_base/2} 0 ${vehicle_height/2}" rpy="0 0 0"/>
