Commit message: update

File: urdf/steering.xacro (robot description, xacro)
@@ -31,5 +31,5 @@
       <inertial>
         <origin xyz="0 0 0" rpy="0 0 0"/>
-        <mass value="1"/>
+        <mass value="10"/>
         <inertia ixx="0.4"  ixy="0"  ixz="0" iyy="0.6" iyz="0" izz="0.4" />
       </inertial>

File: urdf/vehicle.xacro (robot description, xacro)
@@ -16,11 +16,11 @@
     <inertial>
       <origin xyz="${$(arg wheel_base)/2} 0 0" rpy="0 0 0"/>
-      <mass value="1000.0"/>
-      <inertia ixx="1.0" ixy="0.0" ixz="0.0" iyy="1.0" iyz="0.0" izz="1.0"/>
+      <mass value="2000.0"/>
+      <inertia ixx="60.0" ixy="0.0" ixz="0.0" iyy="1000.0" iyz="0.0" izz="1000.0"/>
     </inertial>
     <visual>
       <origin xyz="1.5 0 0.7" rpy="0 0 0"/>
       <geometry>
-        <box size="3.0 0.9 1.4"/>
+        <box size="4.0 2.0 1.4"/>
       </geometry>
     </visual>
@@ -41,5 +41,5 @@
       <origin xyz="0 0 0" rpy="0 0 0"/>
       <mass value="1.0"/>
-      <inertia ixx="1.0" ixy="0.0" ixz="0.0" iyy="1.0" iyz="0.0" izz="1.0"/>
+      <inertia ixx="0.01" ixy="0.0" ixz="0.0" iyy="1.0" iyz="0.0" izz="0.01"/>
     </inertial>
   </link>
@@ -53,5 +53,5 @@
       <origin xyz="0 0 0" rpy="0 0 0"/>
       <mass value="1.0"/>
-      <inertia ixx="1.0" ixy="0.0" ixz="0.0" iyy="1.0" iyz="0.0" izz="1.0"/>
+      <inertia ixx="0.01" ixy="0.0" ixz="0.0" iyy="1.0" iyz="0.0" izz="0.01"/>
     </inertial>
   </link>
@@ -62,24 +62,7 @@
   <xacro:wheel_macro suffix="wheel_right_rear" parent="wheel_rear_base_link" x="0" y="${-1*$(arg wheel_tread)/2}" yaw="${pi}" radius="$(arg wheel_radius)" width="$(arg wheel_width)"/>
   <xacro:wheel_macro suffix="wheel_left_rear" parent="wheel_rear_base_link" x="0" y="${$(arg wheel_tread)/2}" yaw="${0}" radius="$(arg wheel_radius)" width="$(arg wheel_width)"/>
-    <!-- <transmission name="$wheel_left_rear_trans">
-      <type>transmission_interface/SimpleTransmission</type>
-      <joint name="wheel_left_rear_joint">
-        <hardwareInterface>hardware_interface/VelocityJointInterface</hardwareInterface>
-      </joint>
-      <actuator name="wheel_left_rear_motor">
-         <hardwareInterface>hardware_interface/VelocityJointInterface</hardwareInterface>
-         <mechanismReduction>1</mechanismReduction>
-      </actuator>
-    </transmission>
-    <transmission name="wheel_right_rear_trans">
-      <type>transmission_interface/SimpleTransmission</type>
-      <joint name="wheel_right_rear_joint">
-        <hardwareInterface>hardware_interface/VelocityJointInterface</hardwareInterface>
-      </joint>
-      <actuator name="wheel_right_rear_motor">
-         <hardwareInterface>hardware_interface/VelocityJointInterface</hardwareInterface>
-         <mechanismReduction>1</mechanismReduction>
-      </actuator>
-    </transmission> -->
+  <!-- gazebo -->
+ 	<!-- <xacro:include filename="$(find catvehicle)/urdf/wheel.gazebo"/>
+ 	<xacro:include filename="$(find catvehicle)/urdf/steering.gazebo"/> -->
   <gazebo>
     <plugin name="gazebo_ros_control" filename="libgazebo_ros_control.so">

File: urdf/wheel.xacro (robot description, xacro)
@@ -1,6 +1,3 @@
 <robot xmlns:xacro="http://ros.org/wiki/xacro">
-  <material name="black">
-    <color rgba="0.1 0.1 0.1 2.0"/>
-  </material>
   <xacro:property name="pi" value="3.141592" />
   <xacro:macro name="wheel_macro" params="suffix parent x y yaw radius width">
@@ -26,6 +23,6 @@
       <inertial>
         <origin xyz="0 0 0" rpy="0 0 0"/>
-        <mass value="11"/>
-        <inertia ixx="50.0"  ixy="0"  ixz="0" iyy="50.0" iyz="0" izz="100.0" />
+        <mass value="40"/>
+        <inertia ixx="100.0"  ixy="0"  ixz="0" iyy="50.0" iyz="0" izz="50.0" />
       </inertial>
       <collision>

Commit message: update

File: urdf/steering.xacro (robot description, xacro)
@@ -1,4 +1,4 @@
 <robot xmlns:xacro="http://ros.org/wiki/xacro">
-  <xacro:property name="pi" value="3.141592" />
+  <xacro:property name="pi" value="3.1415926835897931" />
   <xacro:macro name="steering_macro" params="suffix parent x y yaw length">
     <joint name="${suffix}_joint" type="revolute">
@@ -9,5 +9,29 @@
       <limit effort="1000.0" lower="-1" upper="1" velocity="0.5"/>
     </joint>
-    <transmission name="${suffix}_trans">
+    <link name="${suffix}_link">
+      <visual>
+        <geometry>
+          <box size="0.01 0.01 0.01"/>
+          <!-- <cylinder length="0.01" radius="0.1"/> -->
+        </geometry>
+        <origin xyz="0 0 0" rpy="0 0 0"/>
+        <material name="black">
+          <color rgba="0.1 0.1 0.1 2.0"/>
+        </material>
+      </visual>
+      <inertial>
+        <origin xyz="0 0 0" rpy="0 0 0"/>
+        <mass value="0.01"/>
+        <inertia ixx="${(0.0001+0.0001)*0.01/12}"  ixy="0"  ixz="0" iyy="${(0.0001+0.0001)*0.01/12}" iyz="0" izz="${(0.0001+0.0001)*0.01/12}" />
+      </inertial>
+      <collision>
+        <origin xyz="0 0 0" rpy="0 0 0"/>
+        <geometry>
+          <box size="0.01 0.01 0.01"/>
+          <!-- <cylinder radius="0.1" length="0.01" /> -->
+        </geometry>
+      </collision>
+    </link>
+    <!-- <transmission name="${suffix}_trans">
       <type>transmission_interface/SimpleTransmission</type>
       <joint name="${suffix}_joint">
@@ -18,22 +42,6 @@
          <mechanismReduction>1</mechanismReduction>
       </actuator>
-    </transmission>
-    <link name="${suffix}_link">
-      <visual>
-        <geometry>
-          <cylinder length="0.01" radius="0.1"/>
-        </geometry>
-        <origin xyz="0 0 0" rpy="0 0 0"/>
-        <material name="black">
-          <color rgba="0.1 0.1 0.1 2.0"/>
-        </material>
-      </visual>
-      <inertial>
-        <origin xyz="0 0 0" rpy="0 0 0"/>
-        <mass value="10"/>
-        <inertia ixx="0.4"  ixy="0"  ixz="0" iyy="0.6" iyz="0" izz="0.4" />
-      </inertial>
-    </link>
-    <gazebo reference="${suffix}_link">
+    </transmission> -->
+    <!-- <gazebo reference="${suffix}_link">
       <material>Gazebo/Red</material>
         <mu1 value="0.6" />
@@ -43,5 +51,5 @@
         <minDepth value="0.01"/>
         <maxVel value="10.0" />
-    </gazebo>
+    </gazebo> -->
   </xacro:macro>
 </robot>

File: urdf/vehicle.xacro (robot description, xacro)
@@ -6,5 +6,10 @@
   <xacro:arg name="wheel_base" default="2.950"/>
   <xacro:arg name="wheel_tread" default="1.55"/>
-  <xacro:property name="pi" value="3.141592" />
+  <xacro:arg name="vehicle_mass" default="5000.0"/>
+  <xacro:arg name="vehicle_length" default="4.82"/>
+  <xacro:arg name="vehicle_width" default="1.81"/>
+  <xacro:arg name="vehicle_height" default="1.5"/>
+  <xacro:arg name="vehicle_mass_height" default="0.5"/>
+  <xacro:property name="pi" value="3.1415926835897931" />
   <link name="base_link"/>
   <joint name="base_joint" type="fixed">
@@ -16,53 +21,35 @@
     <inertial>
       <origin xyz="${$(arg wheel_base)/2} 0 0" rpy="0 0 0"/>
-      <mass value="2000.0"/>
-      <inertia ixx="60.0" ixy="0.0" ixz="0.0" iyy="1000.0" iyz="0.0" izz="1000.0"/>
+      <mass value="$(arg vehicle_mass)"/>
+      <inertia ixx="${($(arg vehicle_width)*$(arg vehicle_width)+$(arg vehicle_mass_height)*$(arg vehicle_mass_height))*$(arg vehicle_mass)/12.0}" ixy="0.0" ixz="0.0"
+               iyy="${($(arg vehicle_length)*$(arg vehicle_length)+$(arg vehicle_mass_height)*$(arg vehicle_mass_height))*$(arg vehicle_mass)/12.0}" iyz="0.0"
+               izz="${($(arg vehicle_width)*$(arg vehicle_width)+$(arg vehicle_length)*$(arg vehicle_length))*$(arg vehicle_mass)/12.0}"/>
     </inertial>
     <visual>
-      <origin xyz="1.5 0 0.7" rpy="0 0 0"/>
+      <origin xyz="${$(arg wheel_base)/2} 0 ${$(arg vehicle_height)/2}" rpy="0 0 0"/>
       <geometry>
-        <box size="4.0 2.0 1.4"/>
+        <box size="$(arg vehicle_length) $(arg vehicle_width) $(arg vehicle_height)"/>
       </geometry>
     </visual>
     <collision>
-      <origin xyz="1.5 0 0.7" rpy="0 0 0"/>
+      <origin xyz="${$(arg wheel_base)/2} 0 ${$(arg vehicle_height)/2}" rpy="0 0 0"/>
       <geometry>
-        <box size="3.0 0.9 1.4"/>
+        <box size="$(arg vehicle_length) 0.9 $(arg vehicle_height)"/>
       </geometry>
     </collision>
   </link>
-  <joint name="wheel_front_base_joint" type="fixed">
-    <parent link="wheel_base_link"/>
-    <origin rpy="0 0 0" xyz="$(arg wheel_base) 0 0"/>
-    <child  link="wheel_front_base_link"/>
-  </joint>
-  <link name="wheel_front_base_link">
-    <inertial>
-      <origin xyz="0 0 0" rpy="0 0 0"/>
-      <mass value="1.0"/>
-      <inertia ixx="0.01" ixy="0.0" ixz="0.0" iyy="1.0" iyz="0.0" izz="0.01"/>
-    </inertial>
-  </link>
-  <joint name="wheel_rear_base_joint" type="fixed">
-    <parent link="wheel_base_link"/>
-    <origin rpy="0 0 0" xyz="0 0 0"/>
-    <child  link="wheel_rear_base_link"/>
-  </joint>
-  <link name="wheel_rear_base_link">
-    <inertial>
-      <origin xyz="0 0 0" rpy="0 0 0"/>
-      <mass value="1.0"/>
-      <inertia ixx="0.01" ixy="0.0" ixz="0.0" iyy="1.0" iyz="0.0" izz="0.01"/>
-    </inertial>
-  </link>
-  <xacro:steering_macro suffix="steering_right_front" parent="wheel_front_base_link" x="0" y="${-1*$(arg wheel_tread)/2}" yaw="0" length="$(arg wheel_width)"/>
-  <xacro:steering_macro suffix="steering_left_front" parent="wheel_front_base_link" x="0" y="${$(arg wheel_tread)/2}" yaw="0" length="$(arg wheel_width)"/>
+  <xacro:steering_macro suffix="steering_right_front" parent="wheel_base_link" x="$(arg wheel_base)" y="${-1*$(arg wheel_tread)/2}" yaw="0" length="$(arg wheel_width)"/>
+  <xacro:steering_macro suffix="steering_left_front" parent="wheel_base_link" x="$(arg wheel_base)" y="${$(arg wheel_tread)/2}" yaw="0" length="$(arg wheel_width)"/>
   <xacro:wheel_macro suffix="wheel_right_front" parent="steering_right_front_link" x="0" y="0" yaw="${pi}" radius="$(arg wheel_radius)" width="$(arg wheel_width)"/>
   <xacro:wheel_macro suffix="wheel_left_front" parent="steering_left_front_link" x="0" y="0" yaw="${0}" radius="$(arg wheel_radius)" width="$(arg wheel_width)"/>
-  <xacro:wheel_macro suffix="wheel_right_rear" parent="wheel_rear_base_link" x="0" y="${-1*$(arg wheel_tread)/2}" yaw="${pi}" radius="$(arg wheel_radius)" width="$(arg wheel_width)"/>
-  <xacro:wheel_macro suffix="wheel_left_rear" parent="wheel_rear_base_link" x="0" y="${$(arg wheel_tread)/2}" yaw="${0}" radius="$(arg wheel_radius)" width="$(arg wheel_width)"/>
+  <!-- <xacro:wheel_macro suffix="wheel_right_front" parent="wheel_base_link" x="$(arg wheel_base)" y="${-1*$(arg wheel_tread)/2}" yaw="${pi}" radius="$(arg wheel_radius)" width="$(arg wheel_width)"/>
+  <xacro:wheel_macro suffix="wheel_left_front" parent="wheel_base_link" x="$(arg wheel_base)" y="${$(arg wheel_tread)/2}" yaw="${0}" radius="$(arg wheel_radius)" width="$(arg wheel_width)"/> -->
+  <xacro:wheel_macro suffix="wheel_right_rear" parent="wheel_base_link" x="0" y="${-1*$(arg wheel_tread)/2}" yaw="${pi}" radius="$(arg wheel_radius)" width="$(arg wheel_width)"/>
+  <xacro:wheel_macro suffix="wheel_left_rear" parent="wheel_base_link" x="0" y="${$(arg wheel_tread)/2}" yaw="${0}" radius="$(arg wheel_radius)" width="$(arg wheel_width)"/>
+  <!-- actuator -->
+ 	<xacro:include filename="$(find vehicle_model)/urdf/actuator.xacro"/>
   <!-- gazebo -->
- 	<!-- <xacro:include filename="$(find catvehicle)/urdf/wheel.gazebo"/>
- 	<xacro:include filename="$(find catvehicle)/urdf/steering.gazebo"/> -->
+ 	<xacro:include filename="$(find vehicle_model)/urdf/wheel.gazebo"/>
+ 	<xacro:include filename="$(find vehicle_model)/urdf/steering.gazebo"/>
   <gazebo>
     <plugin name="gazebo_ros_control" filename="libgazebo_ros_control.so">
@@ -73,5 +60,5 @@
   <gazebo>
     <plugin filename="libgazebo_ros_joint_state_publisher.so" name="joint_state_publisher">
-      <jointName>wheel_left_rear_joint, wheel_right_rear_joint, steering_left_front_joint, steering_right_front_joint, wheel_right_front_joint, wheel_left_front_joint</jointName>
+      <jointName>wheel_left_rear_joint, wheel_right_rear_joint, steering_left_front_joint, steering_right_front_joint</jointName>
       <updateRate>50.0</updateRate>
       <robotNamespace>/autoware</robotNamespace>

File: urdf/wheel.xacro (robot description, xacro)
@@ -1,5 +1,6 @@
 <robot xmlns:xacro="http://ros.org/wiki/xacro">
-  <xacro:property name="pi" value="3.141592" />
+  <xacro:property name="pi" value="3.1415926835897931" />
   <xacro:macro name="wheel_macro" params="suffix parent x y yaw radius width">
+    <xacro:property name="mass" value="40" />
     <joint name="${suffix}_joint" type="continuous">
       <origin rpy="0 0 ${pi/2}" xyz="${x} ${y} 0"/>
@@ -8,5 +9,5 @@
       <axis xyz="1 0 0"/>
       <dynamics damping="0.1"/>
-      <limit effort="10000" velocity="100" />
+      <limit effort="50000" velocity="50" />
       <joint_properties damping="0.0" friction="0.0" />
     </joint>
@@ -23,6 +24,6 @@
       <inertial>
         <origin xyz="0 0 0" rpy="0 0 0"/>
-        <mass value="40"/>
-        <inertia ixx="100.0"  ixy="0"  ixz="0" iyy="50.0" iyz="0" izz="50.0" />
+        <mass value="${mass}"/>
+        <inertia ixx="${mass*radius*radius/2}"  ixy="0"  ixz="0" iyy="${radius*radius*mass/4+width*width*mass/12}" iyz="0" izz="${radius*radius*mass/4+width*width*mass/12}" />
       </inertial>
       <collision>
@@ -33,5 +34,5 @@
       </collision>
     </link>
-    <transmission name="${suffix}_trans">
+    <!-- <transmission name="${suffix}_trans">
       <type>transmission_interface/SimpleTransmission</type>
       <joint name="${suffix}_joint">
@@ -42,14 +43,14 @@
          <mechanismReduction>1</mechanismReduction>
       </actuator>
-    </transmission>
-    <gazebo reference="${suffix}_link">
+    </transmission> -->
+    <!-- <gazebo reference="${suffix}_link">
       <material>Gazebo/Red</material>
-      <mu1 value="1.0" />
-      <mu2 value="1.0" />
-   		<kp value="1000000" />
+      <mu1 value="10000.0" />
+      <mu2 value="10000.0" />
+   		<kp value="100000" />
       <kd value="0.1" />
       <minDepth value="0.01" />
       <maxVel  value="100.0" />
-    </gazebo>
+    </gazebo> -->
   </xacro:macro>
 </robot>

Commit message: update

File: urdf/steering.xacro (robot description, xacro)
@@ -3,4 +3,7 @@
   <xacro:property name="pi" value="3.1415926835897931" />
   <xacro:macro name="steering_macro" params="suffix parent x y yaw length">
+    <xacro:property name="radius" value="0.1" />
+    <xacro:property name="length" value="0.01" />
+    <xacro:property name="mass" value="10.0" />
     <joint name="${suffix}_joint" type="revolute">
       <origin rpy="0 0 0" xyz="${x} ${y} 0"/>
@@ -13,5 +16,5 @@
       <visual>
         <geometry>
-          <cylinder radius="0.1" length="0.01"/>
+          <cylinder radius="${radius}" length="${length}"/>
         </geometry>
         <origin xyz="0 0 0" rpy="${pi/2} 0 0"/>
@@ -22,8 +25,8 @@
       <inertial>
         <origin xyz="0 0 0" rpy="0 0 0"/>
-        <mass value="10.0"/>
-        <inertia ixx="0.0250833"  ixy="0"  ixz="0" iyy="0.05" iyz="0" izz="0.0250833" />
-        <!-- <mass value="10.0"/>
-        <inertia ixx="0.4"  ixy="0"  ixz="0" iyy="0.6" iyz="0" izz="0.4" /> -->
+        <mass value="${mass}"/>
+        <inertia ixx="${radius*radius*mass/4+length*length*mass/12}"  ixy="0"  ixz="0"
+                 iyy="${mass*radius*radius/2}" iyz="0"
+                 izz="${radius*radius*mass/4+length*length*mass/12}" />
       </inertial>
       <!-- <collision>

Commit message: update

File: urdf/steering.xacro (robot description, xacro)
@@ -11,5 +11,5 @@
       <child  link="${suffix}_link"/>
       <axis xyz="0 0 1"/>
-      <limit effort="1000.0" lower="-0.6" upper="0.6" velocity="0.5"/>
+      <limit effort="100000000.0" lower="-0.6" upper="0.6" velocity="0.5"/>
     </joint>
     <link name="${suffix}_link">
