Commit message: update

File: vehicle_model/urdf/body.xacro (robot description, xacro)
@@ -1,6 +1,6 @@
 <?xml version="1.0"?>
 <robot xmlns:xacro="http://ros.org/wiki/xacro">
+  <xacro:macro name="body_macro" params="suffix parent wheel_radius wheel_base vehicle_mass vehicle_mass_height vehicle_width vehicle_length vehicle_height">
   <xacro:property name="pi" value="3.1415926835897931" />
-  <xacro:macro name="body_macro" params="suffix parent wheel_radius wheel_base vehicle_mass vehicle_mass_height vehicle_width vehicle_length vehicle_height">
     <joint name="${suffix}_joint" type="fixed">
       <parent link="${parent}"/>

File: vehicle_model/urdf/steering.xacro (robot description, xacro)
@@ -1,6 +1,6 @@
 <?xml version="1.0"?>
 <robot xmlns:xacro="http://ros.org/wiki/xacro">
-  <xacro:property name="pi" value="3.1415926835897931" />
   <xacro:macro name="steering_macro" params="suffix parent x y yaw length">
+    <xacro:property name="pi" value="3.1415926835897931" />
     <xacro:property name="radius" value="0.1" />
     <xacro:property name="length" value="0.01" />

File: vehicle_model/urdf/vehicle.xacro (robot description, xacro)
@@ -8,41 +8,60 @@
   <xacro:include filename="$(find camera_description)/urdf/monocular_camera.xacro"/>
   <xacro:include filename="$(find imu_description)/urdf/imu.xacro"/>
-  <xacro:arg name="wheel_radius" default="0.341"/>
-  <xacro:arg name="wheel_width" default="0.225"/>
-  <xacro:arg name="wheel_base" default="2.950"/>
-  <xacro:arg name="wheel_tread" default="1.55"/>
-  <xacro:arg name="vehicle_mass" default="5000.0"/>
-  <xacro:arg name="vehicle_length" default="4.82"/>
-  <xacro:arg name="vehicle_width" default="1.81"/>
-  <xacro:arg name="vehicle_height" default="1.5"/>
   <xacro:arg name="gpu" default="false"/>
-  <xacro:arg name="vehicle_mass_height" default="0.5"/>
   <xacro:property name="pi" value="3.1415926835897931"/>
   <link name="base_link"/>
-  <!-- vehicle -->
+  <!-- ================ vehicle ================ -->
+  <!-- load parameter -->
+	<xacro:property name="vehicle_info" value="${load_yaml('$(find vehicle_model)/config/vehicle_info.yaml')}"/>
+  <!-- set parameter -->
+	<xacro:property name="wheel_radius" value="${vehicle_info['wheel_radius']}"/>
+  <xacro:property name="wheel_width" value="${vehicle_info['wheel_width']}"/>
+  <xacro:property name="wheel_base" value="${vehicle_info['wheel_base']}"/>
+  <xacro:property name="wheel_tread" value="${vehicle_info['wheel_tread']}"/>
+  <xacro:property name="vehicle_mass" value="${vehicle_info['vehicle_mass']}"/>
+  <xacro:property name="vehicle_length" value="${vehicle_info['vehicle_length']}"/>
+  <xacro:property name="vehicle_width" value="${vehicle_info['vehicle_width']}"/>
+  <xacro:property name="vehicle_height" value="${vehicle_info['vehicle_height']}"/>
+  <xacro:property name="vehicle_mass_height" value="0.5"/>
   <xacro:body_macro suffix="wheel_base"
                     parent="base_link"
-                    wheel_radius="$(arg wheel_radius)"
-                    wheel_base="$(arg wheel_base)"
-                    vehicle_mass="$(arg vehicle_mass)"
-                    vehicle_mass_height="$(arg vehicle_mass_height)"
-                    vehicle_length="$(arg vehicle_length)"
-                    vehicle_width="$(arg vehicle_width)"
-                    vehicle_height="$(arg vehicle_height)"/>
-  <xacro:steering_macro suffix="steering_right_front" parent="wheel_base_link" x="$(arg wheel_base)" y="${-1*$(arg wheel_tread)/2}" yaw="0" length="$(arg wheel_width)"/>
-  <xacro:steering_macro suffix="steering_left_front" parent="wheel_base_link" x="$(arg wheel_base)" y="${$(arg wheel_tread)/2}" yaw="0" length="$(arg wheel_width)"/>
-  <xacro:wheel_macro suffix="wheel_right_front" parent="steering_right_front_link" x="0" y="0" yaw="${pi}" radius="$(arg wheel_radius)" width="$(arg wheel_width)"/>
-  <xacro:wheel_macro suffix="wheel_left_front" parent="steering_left_front_link" x="0" y="0" yaw="${0}" radius="$(arg wheel_radius)" width="$(arg wheel_width)"/>
-  <xacro:wheel_macro suffix="wheel_right_rear" parent="wheel_base_link" x="0" y="${-1*$(arg wheel_tread)/2}" yaw="${pi}" radius="$(arg wheel_radius)" width="$(arg wheel_width)"/>
-  <xacro:wheel_macro suffix="wheel_left_rear" parent="wheel_base_link" x="0" y="${$(arg wheel_tread)/2}" yaw="${0}" radius="$(arg wheel_radius)" width="$(arg wheel_width)"/>
-  <!-- sensor -->
-  <HDL-32E parent="base_link" name="velodyne" topic="/velodyne_points" hz="10" samples="220" gpu="$(arg gpu)">
-    <origin xyz="0 0 2.0" rpy="0 0 0" />
-  </HDL-32E>
-  <xacro:monocular_camera_macro suffix="camera" parent="base_link" namespace="" x="0" y="0" z="2.5" roll="0" pitch="0" yaw="0"  fps="30" width="800" height="400" fov="1.3"/>
-  <xacro:imu_macro suffix="imu" parent="base_link" namespace="" x="0" y="0" z="2.6" roll="0" pitch="0" yaw="0"  fps="100" />
+                    wheel_radius="${wheel_radius}"
+                    wheel_base="${wheel_base}"
+                    vehicle_mass="${vehicle_mass}"
+                    vehicle_mass_height="${vehicle_mass_height}"
+                    vehicle_length="${vehicle_length}"
+                    vehicle_width="${vehicle_width}"
+                    vehicle_height="${vehicle_height}"/>
+  <xacro:steering_macro suffix="steering_right_front" parent="wheel_base_link" x="${wheel_base}" y="${-1*wheel_tread/2}" yaw="0" length="${wheel_width}"/>
+  <xacro:steering_macro suffix="steering_left_front" parent="wheel_base_link" x="${wheel_base}" y="${wheel_tread/2}" yaw="0" length="${wheel_width}"/>
+  <xacro:wheel_macro suffix="wheel_right_front" parent="steering_right_front_link" x="0" y="0" yaw="${pi}" radius="${wheel_radius}" width="${wheel_width}"/>
+  <xacro:wheel_macro suffix="wheel_left_front" parent="steering_left_front_link" x="0" y="0" yaw="0" radius="${wheel_radius}" width="${wheel_width}"/>
+  <xacro:wheel_macro suffix="wheel_right_rear" parent="wheel_base_link" x="0" y="${-1*wheel_tread/2}" yaw="${pi}" radius="${wheel_radius}" width="${wheel_width}"/>
+  <xacro:wheel_macro suffix="wheel_left_rear" parent="wheel_base_link" x="0" y="${wheel_tread/2}" yaw="0" radius="${wheel_radius}" width="${wheel_width}"/>
   <!-- actuator -->
  	<xacro:include filename="$(find vehicle_model)/urdf/actuator.xacro"/>
   <!-- gazebo -->
  	<xacro:include filename="$(find vehicle_model)/urdf/vehicle.gazebo"/>
+  <!-- ================ sensor ================ -->
+	<xacro:property name="calibration" value="${load_yaml('$(find vehicle_model)/config/calibration.yaml')}"/>
+  <HDL-32E parent="base_link" name="velodyne" topic="/velodyne_points" hz="10" samples="220" gpu="$(arg gpu)">
+    <origin xyz="${calibration['base_link2velodyne']['x']} ${calibration['base_link2velodyne']['y']} ${calibration['base_link2velodyne']['z']}"
+            rpy="${calibration['base_link2velodyne']['roll']} ${calibration['base_link2velodyne']['pitch']} ${calibration['base_link2velodyne']['yaw']}" />
+  </HDL-32E>
+  <xacro:monocular_camera_macro suffix="camera" parent="base_link" namespace=""
+                                x="${calibration['base_link2camera']['x']}"
+                                y="${calibration['base_link2camera']['y']}"
+                                z="${calibration['base_link2camera']['z']}"
+                                roll="${calibration['base_link2camera']['roll']}"
+                                pitch="${calibration['base_link2camera']['pitch']}"
+                                yaw="${calibration['base_link2camera']['yaw']}"
+                                fps="30" width="800" height="400" fov="1.3"/>
+  <xacro:imu_macro suffix="imu" parent="base_link" namespace=""
+                   x="${calibration['base_link2imu']['x']}"
+                   y="${calibration['base_link2imu']['y']}"
+                   z="${calibration['base_link2imu']['z']}"
+                   roll="${calibration['base_link2imu']['roll']}"
+                   pitch="${calibration['base_link2imu']['pitch']}"
+                   yaw="${calibration['base_link2imu']['yaw']}"
+                   fps="100" />
 </robot>

File: vehicle_model/urdf/wheel.xacro (robot description, xacro)
@@ -1,6 +1,6 @@
 <?xml version="1.0"?>
 <robot xmlns:xacro="http://ros.org/wiki/xacro">
-  <xacro:property name="pi" value="3.1415926835897931" />
   <xacro:macro name="wheel_macro" params="suffix parent x y yaw radius width">
+    <xacro:property name="pi" value="3.1415926835897931" />
     <xacro:property name="mass" value="40" />
     <joint name="${suffix}_joint" type="continuous">

Commit message: update

File: vehicle_model/urdf/body.xacro (robot description, xacro)
@@ -17,5 +17,9 @@
       </inertial>
       <visual>
-        <origin xyz="${wheel_base/2} 0 ${vehicle_height/2}" rpy="0 ${-pi/2} ${pi/2}"/>
+        <origin xyz="${wheel_base/2} 0 ${vehicle_height/2}" rpy="0 0 0"/>
+        <geometry>
+          <box size="${vehicle_length} 0.9 ${vehicle_height}"/>
+        </geometry>
+        <!-- <origin xyz="${wheel_base/2} 0 ${vehicle_height/2}" rpy="0 ${-pi/2} ${pi/2}"/>
         <geometry>
           <mesh filename="package://vehicle_model/dae/banana.dae" scale="0.7 0.7 0.7"/>
@@ -23,15 +27,6 @@
         <material name="black">
             <color rgba="0.1 0.1 0.1 2.0"/>
-        </material>
+        </material> -->
       </visual>
-      <!-- <visual>
-        <origin xyz="${wheel_base/2} 0 ${vehicle_height/2}" rpy="0 0 0"/>
-        <geometry>
-          <box size="${vehicle_length} ${vehicle_width} ${vehicle_height}"/>
-        </geometry>
-        <material name="black">
-            <color rgba="0.1 0.1 0.1 2.0"/>
-        </material>
-      </visual> -->
       <collision>
         <origin xyz="${wheel_base/2} 0 ${vehicle_height/2}" rpy="0 0 0"/>

File: vehicle_model/urdf/wheel.xacro (robot description, xacro)
@@ -15,8 +15,12 @@
     <link name="${suffix}_link">
       <visual>
+        <origin xyz="0 0 0" rpy="0 ${pi/2} 0"/>
         <geometry>
+          <cylinder radius="${radius}" length="${width}" />
+        </geometry>
+        <!-- <geometry>
           <mesh filename="package://vehicle_model/dae/wheel.dae" scale="${0.01173*radius} ${0.01173*radius} ${0.01173*radius}"/>
         </geometry>
-        <origin xyz="0 0 0" rpy="0 0 ${yaw}"/>
+        <origin xyz="0 0 0" rpy="0 0 ${yaw}"/> -->
         <material name="black">
           <color rgba="0.1 0.1 0.1 2.0"/>

Commit message: update

File: vehicle_model/urdf/body.xacro (robot description, xacro)
@@ -17,15 +17,16 @@
       </inertial>
       <visual>
-        <origin xyz="${wheel_base/2} 0 ${vehicle_height/2}" rpy="0 0 0"/>
+        <!-- <origin xyz="${wheel_base/2} 0 ${vehicle_height/2}" rpy="0 0 0"/>
         <geometry>
           <box size="${vehicle_length} 0.9 ${vehicle_height}"/>
-        </geometry>
-        <!-- <origin xyz="${wheel_base/2} 0 ${vehicle_height/2}" rpy="0 ${-pi/2} ${pi/2}"/>
+        </geometry> -->
+        <!-- <origin xyz="${wheel_base/2} 0 ${vehicle_height/2}" rpy="0 ${-pi/2} ${pi/2}"/> -->
+        <origin xyz="0 0 0" rpy="0 0 0"/>
         <geometry>
-          <mesh filename="package://vehicle_model/dae/banana.dae" scale="0.7 0.7 0.7"/>
+          <mesh filename="package://vehicle_model/dae/body.dae" scale="${wheel_base/2.85} 1 1"/>
         </geometry>
         <material name="black">
-            <color rgba="0.1 0.1 0.1 2.0"/>
-        </material> -->
+            <color rgba="0.1 0.1 0.1 0.5"/>
+        </material>
       </visual>
       <collision>

File: vehicle_model/urdf/wheel.xacro (robot description, xacro)
@@ -15,13 +15,9 @@
     <link name="${suffix}_link">
       <visual>
-        <origin xyz="0 0 0" rpy="0 ${pi/2} 0"/>
         <geometry>
-          <cylinder radius="${radius}" length="${width}" />
+          <mesh filename="package://vehicle_model/dae/wheel.dae" scale="${3*radius} ${3*radius} ${3*radius}"/>
         </geometry>
-        <!-- <geometry>
-          <mesh filename="package://vehicle_model/dae/wheel.dae" scale="${0.01173*radius} ${0.01173*radius} ${0.01173*radius}"/>
-        </geometry>
-        <origin xyz="0 0 0" rpy="0 0 ${yaw}"/> -->
-        <material name="black">
+        <origin xyz="0 0 0" rpy="0 0 ${yaw}"/>
+        <material name="gray">
           <color rgba="0.1 0.1 0.1 2.0"/>
         </material>
