Commit message: change constitution

File: vehicle/vehicle_model/urdf/body.xacro (robot description, xacro)
@@ -24,5 +24,5 @@
         <origin xyz="0 0 0" rpy="0 0 0"/>
         <geometry>
-          <mesh filename="package://vehicle_model/dae/body.dae" scale="${wheel_base/2.85} 1 1"/>
+          <mesh filename="package://vehicle_model/mesh/body.dae" scale="${wheel_base/2.85} 1 1"/>
         </geometry>
         <material name="black">

File: vehicle/vehicle_model/urdf/steering.xacro (robot description, xacro)
@@ -38,3 +38,13 @@
     </link>
   </xacro:macro>
+  <xacro:macro name="steering_link_macro" params="suffix parent x y">
+    <xacro:property name="pi" value="3.1415926835897931" />
+    <joint name="${suffix}_joint" type="fixed">
+      <origin rpy="0 0 0" xyz="${x} ${y} 0"/>
+      <parent link="${parent}"/>
+      <child  link="${suffix}_link"/>
+    </joint>
+    <link name="${suffix}_link">
+    </link>
+  </xacro:macro>
 </robot>

File: vehicle/vehicle_model/urdf/vehicle.xacro (robot description, xacro)
@@ -10,5 +10,5 @@
   <xacro:arg name="gpu" default="false"/>
   <xacro:property name="pi" value="3.1415926835897931"/>
-  <link name="base_link"/>
+  <link name="base_footprint"/>
   <!-- ================ vehicle ================ -->
   <!-- load parameter -->
@@ -24,6 +24,7 @@
   <xacro:property name="vehicle_height" value="${vehicle_info['vehicle_height']}"/>
   <xacro:property name="vehicle_mass_height" value="0.5"/>
-  <xacro:body_macro suffix="wheel_base"
-                    parent="base_link"
+  <!-- body-->
+  <xacro:body_macro suffix="base"
+                    parent="base_footprint"
                     wheel_radius="${wheel_radius}"
                     wheel_base="${wheel_base}"
@@ -33,10 +34,13 @@
                     vehicle_width="${vehicle_width}"
                     vehicle_height="${vehicle_height}"/>
-  <xacro:steering_macro suffix="steering_right_front" parent="wheel_base_link" x="${wheel_base}" y="${-1*wheel_tread/2}" yaw="0" length="${wheel_width}"/>
-  <xacro:steering_macro suffix="steering_left_front" parent="wheel_base_link" x="${wheel_base}" y="${wheel_tread/2}" yaw="0" length="${wheel_width}"/>
+  <!-- steering-->
+  <xacro:steering_link_macro suffix="steering_front" parent="base_link" x="${wheel_base}" y="0"/>
+  <xacro:steering_macro suffix="steering_right_front" parent="steering_front_link" x="0" y="${-1*wheel_tread/2}" yaw="0" length="${wheel_width}"/>
+  <xacro:steering_macro suffix="steering_left_front" parent="steering_front_link" x="0" y="${wheel_tread/2}" yaw="0" length="${wheel_width}"/>
+  <!-- wheel -->
   <xacro:wheel_macro suffix="wheel_right_front" parent="steering_right_front_link" x="0" y="0" yaw="${pi}" radius="${wheel_radius}" width="${wheel_width}"/>
   <xacro:wheel_macro suffix="wheel_left_front" parent="steering_left_front_link" x="0" y="0" yaw="0" radius="${wheel_radius}" width="${wheel_width}"/>
-  <xacro:wheel_macro suffix="wheel_right_rear" parent="wheel_base_link" x="0" y="${-1*wheel_tread/2}" yaw="${pi}" radius="${wheel_radius}" width="${wheel_width}"/>
-  <xacro:wheel_macro suffix="wheel_left_rear" parent="wheel_base_link" x="0" y="${wheel_tread/2}" yaw="0" radius="${wheel_radius}" width="${wheel_width}"/>
+  <xacro:wheel_macro suffix="wheel_right_rear" parent="base_link" x="0" y="${-1*wheel_tread/2}" yaw="${pi}" radius="${wheel_radius}" width="${wheel_width}"/>
+  <xacro:wheel_macro suffix="wheel_left_rear" parent="base_link" x="0" y="${wheel_tread/2}" yaw="0" radius="${wheel_radius}" width="${wheel_width}"/>
   <!-- actuator -->
  	<xacro:include filename="$(find vehicle_model)/urdf/actuator.xacro"/>

File: vehicle/vehicle_model/urdf/wheel.xacro (robot description, xacro)
@@ -16,5 +16,5 @@
       <visual>
         <geometry>
-          <mesh filename="package://vehicle_model/dae/wheel.dae" scale="${3*radius} ${3*radius} ${3*radius}"/>
+          <mesh filename="package://vehicle_model/mesh/wheel.dae" scale="${3*radius} ${3*radius} ${3*radius}"/>
         </geometry>
         <origin xyz="0 0 0" rpy="0 0 ${yaw}"/>
